File: project.brd (EAGLE design)
At the start: 48.3 x 66 mm, 32 parts, among them J2 AUDIO_JACK_3.5MM_KIT, J3 AUDIO_JACK_3.5MM_KIT, J4 AUDIO_JACK_3.5MM_KIT, U1 TL081N, U2 TL081N, X1 736880-49, X2 736880-49

Commit message: Fixing all bugs thus far that were in the schematic. PCB layout now broken!
Parts:
- added C12: 10uF, resistor:CT6032
- added IC1: LM1117LD-3.3, lm1117_11:WSON8-4X4
- added R1, R10, R13, R14, R17, R18: 3.3k, resistor:0204/5
- added R15, R16: 330, resistor:0204/5
- C11, C4: device rcl:C050-024X044 -> SparkFun-Capacitors:CPOL-RADIAL-2.5MM-5MM
- U1, U2: value TL081N -> TL071
- X1, X2: value 736880-49 -> CONRAD_736880-49; device con-conrad:736880-49 -> JRS:CINCH
- moved C11 120.5 mm to (-12.7, -39.4), turned to 0 degrees
- moved X1 117.9 mm to (-2.54, -64.8), turned to 0 degrees
- moved C4 83.6 mm to (-6.35, -39.4), turned to 0 degrees
- moved X2 75.6 mm to (10.2, -8.89), turned to 0 degrees
Connections:
- removed net N$25: C11.2, X2.1, X2.1@1, X2.1@2
- removed net VBUS: C1.1, J1.VBUS, L1.1
- new net N$1: C4.2, X1.1
- new net N$11: C1.1, C12.-, IC1.2, IC1.3, IC1.4, J1.VBUS
- new net N$2: C4.1, R15.2
- new net N$3: C11.2, X2.2
- new net N$7: IC1.5, IC1.6, IC1.7, IC1.EXP, L1.1
- net GND: now also C12.+, IC1.1, R1.2, R10.2, R13.1, R14.1, R17.2, R18.2, X2.1; no longer X2.2
- net N$10: now also R17.1
- net N$12: now also R10.1
- net N$13: now also R18.1
- net N$14: now also R14.2
- net N$15: now also R13.2
- net N$24: now also R16.1; no longer C11.1
- net N$5: now also R15.1; no longer C4.1
- net N$6: now also C11.1, R16.2; no longer C4.2, X1.1, X1.1@1, X1.1@2
- net N$8: now also R1.1
Routing:
- net N$25: track 51.2 -> 0.00 mm
- net N$6: track 31.3 -> 0.00 mm
- net VBUS: track 10.5 -> 0.00 mm, vias 1 -> 0
- net VCC: track 81.7 -> 76.6 mm
- net GND: track 17.9 -> 12.8 mm
- net N$5: track 27.3 -> 23.5 mm
- net N$24: track 20.4 -> 16.8 mm

Commit message: Updating with new power supply Rev.
Parts:
- added C13: 10u Tantal, resistor:E2-4
- added C14: 470p, resistor:C050-024X044
- added C15: 10p, resistor:C050-024X044
- added C16: 47u, resistor:E2,5-5
- added D1: 1N5819, diode:DO41-10
- added IC2: 78L15Z, linear:TO92
- added L2: Recht groß, inductors:82114R
- added LED1: (no value), led:LED5MM
- added R19: 3.3k, resistor:0207/7
- added R20, R21, R22, R23: ???, resistor:0207/7
- C12: value 10uF -> 100u; device resistor:CT6032 -> resistor:E2,5-5
- C3: value 10uF -> 10u
- IC1: value LM1117LD-3.3 -> ON MC34063A; device lm1117_11:WSON8-4X4 -> mc34063:DIL08
- L1: value Ferrite bead -> 47uH; device inductors:MMICC7 -> inductors:MCC10
- moved L1 163.7 mm to (-16.5, -83.8)
- moved C12 62.9 mm to (-27.9, -138.4)
- moved IC1 27.4 mm to (-15.2, -94.0)
Connections:
- new net N$22: C1.2, C13.+, IC2.1, L1.1, LED1.A
- new net N$23: C12.+, C14.2, D1.C, IC2.3, R20.1
- new net N$25: LED1.K, R19.2
- new net N$26: C15.2, IC1.3
- new net N$28: IC1.5, R20.2, R21.1
- new net N$29: C16.+, IC1.6, J1.VBUS, R22.1
- new net N$31: IC1.7, L2.1, R22.2, R23.1
- net GND: now also C1.1, C12.-, C13.-, C14.1, C15.1, C16.-, IC1.2, IC1.4, IC2.2, R19.1, R21.2; no longer C1.2, C12.+, IC1.1
- net N$11: now also D1.A, IC1.1, L2.2; no longer C1.1, C12.-, IC1.2, IC1.3, IC1.4, J1.VBUS
- net N$7: now also IC1.8, R23.2; no longer IC1.5, IC1.6, IC1.7, IC1.EXP, L1.1
Routing:
- net GND: track 12.8 -> 11.2 mm, vias 1 -> 0

Commit message: Updating to latest prototype revision.
Parts:
- removed C15: 10p, resistor:C050-024X044
- removed C16: 47u, resistor:E2,5-5
- removed R16: 330, resistor:0204/5
- removed R17: 3.3k, resistor:0204/5
- removed R20, R21, R22, R23: ???, resistor:0207/7
- removed TPOTL, TPOTR: 100k, pot:B25P
- added TRIM_L, TRIM_R: 100k, pot:B25P
- C1: value 10n -> 47u; device resistor:C050-024X044 -> resistor:E2,5-5
- C10, C7, C8, C9: value 10uF -> 10u; device rcl:C050-024X044 -> resistor:E2-4
- C11: value 1uF -> 10u; device SparkFun-Capacitors:CPOL-RADIAL-2.5MM-5MM -> resistor:E2-4
- C12: value 100u -> 10u; device resistor:E2,5-5 -> resistor:E2-4
- C13: value 10u Tantal -> 100u
- C14: value 470p -> 100u; device resistor:C050-024X044 -> resistor:E2-4
- C2: value 100n -> 10p
- C3: value 10u -> 470p; device resistor:E2,5-5 -> resistor:C050-024X044
- C4: value 1uF -> 100u; device SparkFun-Capacitors:CPOL-RADIAL-2.5MM-5MM -> resistor:E2,5-5
- C5: value 10uF -> 10u Tantal; device rcl:C050-024X044 -> resistor:E2-4
- C6: value 10uF -> 10n; device rcl:C050-024X044 -> resistor:C050-024X044
- L1: value 47uH -> ~20 windings around 4mm ferrite core; device inductors:MCC10 -> inductors:82114R
- L2: value Recht groß -> 47uH; device inductors:82114R -> inductors:MCC10
- R1: value 3.3k -> 180; device resistor:0204/5 -> resistor:0207/7
- R10: value 3.3k -> 22k
- R11: value 10k -> 22k
- R13, R14: value 3.3k -> 10k
- R15: value 330 -> 10k
- R18: value 3.3k -> 330
- R19: value 3.3k -> 330; device resistor:0207/7 -> resistor:0204/5
- R2: value 10k -> 1.2; device resistor:0204/5 -> resistor:0207/7
- R3: value 10k -> 1k; device resistor:0204/5 -> resistor:0207/7
- R4: value 22k -> 15k; device resistor:0204/5 -> resistor:0207/7
- R5: value 22k -> 3.3k; device resistor:0204/5 -> resistor:0207/7
- moved C14 250.4 mm to (34.3, 97.8), turned to 90 degrees
- moved C12 241.4 mm to (21.6, 97.8), turned to 90 degrees
- moved D1 233.4 mm to (21.6, 97.8), turned to 90 degrees
- moved L2 227.0 mm to (24.1, 100.3)
- moved LED1 222.1 mm to (33.0, 97.8), turned to 90 degrees
- moved C13 215.0 mm to (27.9, 97.8), turned to 90 degrees
- moved IC2 203.0 mm to (17.8, 96.5), turned to 90 degrees
- moved IC1 197.1 mm to (8.89, 101.6), turned to 90 degrees
- moved R19 191.0 mm to (26.7, 59.7), turned to 270 degrees
- moved L1 186.8 mm to (40.6, 94.0), turned to 90 degrees
- moved C11 150.9 mm to (44.5, 100.3), turned to 90 degrees
- moved C4 139.2 mm to (29.2, 95.2), turned to 90 degrees
- moved R1 115.8 mm to (26.7, 94.0), turned to 90 degrees
- moved X1 107.4 mm to (44.5, 31.8), turned to 180 degrees
- moved R15 92.5 mm to (34.3, 49.5), turned to 90 degrees
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Connections:
- new net N$33: R11.2, R7.2, R9.2, TRIM_R.E, U2.2
- net GND: now also C1.-, C3.1, C4.-, C5.-, C6.1, R15.1, R3.2, R5.1, X2.2; no longer C1.1, C12.-, C13.-, C14.1, C15.1, C16.-, C3.-, J1.GND, R1.2, R10.2, R11.1, R14.1, R17.2, R18.2, R19.1, R2.1, R21.2, X2.1
- net N$1: now also C13.-; no longer C4.2
- net N$10: now also C8.+, J2.TIP; no longer C6.1, J3.RING, R17.1
- net N$11: now also L1.2; no longer L2.2
- net N$12: now also R10.2, R6.2, R8.2, TRIM_L.E, U1.2; no longer C7.1, J2.TIP, R10.1
- net N$13: now also C8.-, R7.1; no longer C8.1, J3.TIP, R18.1
- net N$14: now also C9.+, J3.RING; no longer C9.1, J4.RING, R14.2
- net N$15: now also C9.-, R8.1; no longer C10.1, J4.TIP, R13.2
- net N$16: now also C10.+, J3.TIP; no longer C5.2, R4.1
- net N$17: now also C10.-, R9.1; no longer C7.2, R5.1
- net N$18: now also C11.+, J4.RING; no longer C6.2, R6.1
- net N$19: now also C11.-, R10.1; no longer C8.2, R7.1
- net N$2: now also C13.+, R18.2; no longer C4.1, R15.2
- net N$20: now also C12.+, J4.TIP; no longer C9.2, R8.1
- net N$21: now also C12.-, R11.1; no longer C10.2, R9.1
- net N$22: now also C5.+, C6.2, L2.1; no longer C1.2, C13.+, L1.1
- net N$23: now also C3.2, C4.+, R4.1; no longer C12.+, C14.2, R20.1
- net N$24: now also R19.1, TRIM_R.S; no longer R16.1, TPOTR.S
- net N$25: now also R5.2; no longer R19.2
- net N$26: now also C2.2; no longer C15.2
- net N$27: now also R14.1, R15.2; no longer R11.2, R12.1
- net N$28: now also R3.1, R4.2; no longer R20.2, R21.1
- net N$29: now also C1.+, R2.1; no longer C16.+, R22.1
- net N$3: now also C14.-, X2.1; no longer C11.2, X2.2
- net N$30: now also J1.GND; no longer R5.2, R7.2, R9.2, TPOTR.E, U2.2
- net N$31: now also L1.1, R1.1, R2.2; no longer L2.1, R22.2, R23.1
- net N$4: now also C7.-, R6.1; no longer R4.2, R6.2, R8.2, TPOTL.E, U1.2
- net N$5: now also R18.1, TRIM_L.S; no longer R15.1, TPOTL.S
- net N$6: now also C14.+, R19.2; no longer C11.1, R16.2
- net N$7: now also R1.2; no longer R23.2
- net N$8: now also C7.+; no longer C5.1, R1.1
- net N$9: now also R12.1, R13.2; no longer R2.2, R3.1
- net VCC: now also L2.2, R14.2; no longer C2.2, C3.+, L1.2, R3.2
Routing:
- net N$30: track 108.0 -> 0.00 mm
- net N$4: track 102.3 -> 0.00 mm
- net VCC: track 76.6 -> 22.1 mm
- net N$33: track 0.00 -> 51.7 mm
- net N$12: track 5.17 -> 56.0 mm
- net GND: track 11.2 -> 0.00 mm
- net N$13: track 5.17 -> 0.00 mm
- net N$10: track 5.17 -> 0.00 mm
- net N$15: track 5.17 -> 0.00 mm
- net N$14: track 5.17 -> 0.00 mm
- net N$21: track 2.54 -> 0.00 mm
- net N$20: track 2.54 -> 0.00 mm
- net N$19: track 2.54 -> 0.00 mm
- net N$18: track 2.54 -> 0.00 mm
- net N$17: track 2.54 -> 0.00 mm
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Other:
- board size 48.3 x 66 mm -> 48.3 x 107.9 mm

Commit message: Re-doing the PCB.
Parts:
- moved C12 62.0 mm to (45.7, 40.6)
- moved C8 61.0 mm to (12.7, 40.6)
- moved C9 61.0 mm to (19.1, 40.6)
- moved C10 60.3 mm to (29.2, 40.6)
- moved C11 60.3 mm to (35.6, 40.6)
- moved C7 58.6 mm to (2.54, 40.6)
- moved R18 54.7 mm to (61.0, 62.2)
- moved C14 52.9 mm to (61.0, 52.1), turned to 0 degrees
- moved U1 52.6 mm to (52.1, 57.1), turned to 0 degrees
- moved C6 48.4 mm to (8.89, 53.3), turned to 0 degrees
- moved TRIM_L 47.6 mm to (52.1, 67.3)
- moved C4 45.8 mm to (3.81, 57.1)
- moved C13 44.1 mm to (61.0, 68.6), turned to 0 degrees
- moved L2 43.5 mm to (29.2, 57.1)
- moved C3 43.1 mm to (25.4, 53.3), turned to 180 degrees
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Routing:
- net N$23: track 0.00 -> 56.9 mm
- net VCC: track 22.1 -> 71.2 mm
- net N$22: track 0.00 -> 39.8 mm, vias 0 -> 1
- net N$29: track 0.00 -> 36.5 mm
- net N$31: track 0.00 -> 36.3 mm, vias 0 -> 2
- net N$28: track 0.00 -> 22.3 mm
- net N$11: track 0.00 -> 22.3 mm
- net N$12: track 56.0 -> 71.8 mm
- net N$3: track 0.00 -> 15.2 mm
- net N$1: track 0.00 -> 15.2 mm
- net N$33: track 51.7 -> 60.5 mm
- net N$9: track 19.6 -> 12.5 mm
- net N$24: track 16.8 -> 9.72 mm
- net N$5: track 23.5 -> 17.1 mm
- net N$20: track 0.00 -> 5.42 mm
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Other:
- board size 48.3 x 107.9 mm -> 82.1 x 48.2 mm
- board text added: "J. R. Schmid • 2018-09-24 • Rev. 8"
- board text removed: "3-WAY HI-FI DISTRIBUTOR"
- board text removed: "J. R. Schmid · 2018-07-22 · Rev. 7"
- board text removed: "The Three Musketeers"
